File: board/BLDC_4.kicad_pcb (KiCad board)
At the start: 4 copper layers, 38.5 x 65 mm, 127 parts, among them K1 SERVO, P1 HALL/Encoder, P101 CANBUS, P2 SWD, P3 PWR_COMM, P4 IN+, P5 IN-, P6 MOTOR1, P7 MOTOR2, P9 MOTOR3, Q1 IRFS7530, Q2 IRFS7530, Q3 IRFS7530, Q4 IRFS7530, Q5 IRFS7530, Q6 IRFS7530, U1 STM32F40X_LQFP64, U2 TC2117, U3 DRV8302, U401 SN65HVD232, X1 MINI-USB-SHIELD-32005-201, X2 8MHz 10ppm

Commit message: - changed some more Vcc labels to +3V3 - combined all input connectors into one big connector - changed can transceiver to MAX3051 - removed HV pin from power connector -> divider now on PS board - updated components - startet layout
Parts:
- removed 1PIN (x2): P***, 1pin
- removed 1PIN (x2): P***, Connect:1pin
- removed C24, C26, C401, C41, C52: 2.2u, CRF1:SMD-0603_c
- removed C25, C33: 100u, w_smd_cap:c_tant_B
- removed C27: 100n, CRF1:SMD-0603_c
- removed C28, C29, C30: 220n, CRF1:SMD-0603_c
- removed C34, C36: 2.2n, CRF1:SMD-0603_c
- removed C37: 15u,100V, w_smd_cap:c_2220
- removed C39, C40, C43, C44, C49: 10u,50V, CRF1:SMD-1206
- removed C51: 15u, 100v, w_smd_cap:c_2220
- removed D4: DIODESCH, Diodes_SMD:SMA_Handsoldering
- removed D5: TVS 5V, w_smd_diode:do214ac
- removed G***: oshw_silkscreen-back_3mm, oshw_silkscreen-back_3mm
- removed K1: SERVO, CRF1:pinhead-1X03
- removed L1: 22u, w_smd_inductors:inductor_smd_8x5mm
- removed P101: CANBUS, JST conn:b4b-ph-kl
- removed P5: IN-, CRF1:1PAD_4x5mm
- removed P6: MOTOR1, CRF1:1PAD_4x5mm
- removed P7: MOTOR2, CRF1:1PAD_4x5mm
- removed P9: MOTOR3, CRF1:1PAD_4x5mm
- removed Q1, Q2, Q3, Q4, Q5, Q6: IRFS7530, CRF1:D2PAK-7-GDS
- removed R1: NTC 10k, CRF1:SMD-0603_r
- removed R17: 18k, CRF1:SMD-0603_r
- removed R18: 3k3, CRF1:SMD-0603_r
- removed R19: 15k, CRF1:SMD-0603_r
- removed R2, R20, R402: 10k, CRF1:SMD-0603_r
- removed R21: 220k, CRF1:SMD-0603_r
- removed R23, R26, R30, R32, R36, R46: 39k, CRF1:SMD-0603_r
- removed R24, R27, R33, R4: 2k2, CRF1:SMD-0603_r
- removed R25: 1M, CRF1:SMD-0603_r
- removed R28, R29, R34, R35, R42, R43: 4R7, CRF1:SMD-0603_r
- removed R401: NI, CRF1:SMD-0603_r
- removed R48, R49, R50, R51: 100R, CRF1:SMD-0603_r
- removed R53, R54: SHUNT, CRF1:WSLP2726
- removed R6: 0R, CRF1:SMD-0603_r
- removed U3: DRV8302, CRF1:TSSOP-56-PP
- removed U401: SN65HVD232, CRF1:SOIC-8-W
- removed X1: MINI-USB-SHIELD-32005-201, CRF1:USB-UX60R-MB-5ST
- added IC1: MAX3051, Housings_SOIC:SOIC-8_3.9x4.9mm_Pitch1.27mm, F.Cu at (187.0, 30.0)
- added REF**: EuroBoard_halb_Type-I_100mmX80mm_holes, EuroBoard_Outline:EuroBoard_halb_Type-I_100mmX80mm_holes, F.Cu at (-209.2, 156.8)
- C1, C8: value 10u,50V -> 100n; footprint CRF1:SMD-1206 -> Capacitors_SMD:C_0805
- C10, C11, C12, C13, C35: footprint CRF1:SMD-0603_c -> Capacitors_SMD:C_0805
- C14, C15, C16, C17, C2, C3, C31, C32, C38, C4, C5, C6, C7: footprint CRF1:SMD-0603_c -> Capacitors_SMD:C_0805; moved to F.Cu
- C18: value 2.2u -> 2u2; footprint CRF1:SMD-0603_c -> Capacitors_SMD:C_0805; moved to F.Cu
- C19: value 120p -> 1n; footprint CRF1:SMD-0603_c -> Capacitors_SMD:C_0805
- C20: value 2.2u -> 1n; footprint CRF1:SMD-0603_c -> Capacitors_SMD:C_0805; moved to F.Cu
- C21: value 6.8n -> 1n; footprint CRF1:SMD-0603_c -> Capacitors_SMD:C_0805
- C22: value 22n -> 1n; footprint CRF1:SMD-0603_c -> Capacitors_SMD:C_0805
- C23: value 2.2u -> 1n; footprint CRF1:SMD-0603_c -> Capacitors_SMD:C_0805
- C9: value 10u,50V -> 100n; footprint CRF1:SMD-1206 -> Capacitors_SMD:C_0805; moved to F.Cu
- D1, D2, D3: footprint LEDs:LED-0603 -> LEDs:LED_0805; moved to F.Cu
- P1: value HALL/Encoder -> Interface; footprint CRF1:MICRO_JST_6 -> Pin_Headers:Pin_Header_Straight_2x10; moved to B.Cu
- P2: footprint CRF1:MICRO_JST_6 -> Pin_Headers:Pin_Header_Straight_2x03; moved to B.Cu
- P3: value PWR_COMM -> USB_B; footprint CRF1:b7b-ph-kl -> alexmod:USBB_vert
- P4: value IN+ -> Power; footprint CRF1:1PAD_4x5mm -> Pin_Headers:Pin_Header_Straight_2x20
- R10, R11, R12, R13, R22, R37, R38, R5, R7, R8, R9: footprint CRF1:SMD-0603_r -> Resistors_SMD:R_0805; moved to F.Cu
- R103, R104: footprint CRF1:SMD-0603_r -> Resistors_SMD:R_0805
- R3: value 39k -> 120R; footprint CRF1:SMD-0603_r -> Resistors_SMD:R_0805; moved to F.Cu
- U1: footprint CRF1:lqfp64_pad_mod -> Housings_QFP:LQFP-64_10x10mm_Pitch0.5mm
- U2: value TC2117 -> AP1117D33; footprint CRF1:SOT-223 -> TO_SOT_Packages_SMD:SOT-223; moved to F.Cu
- X2: footprint CRF1:Crystal_5x3mm -> Crystals:Crystal_HC49-U_Vertical
- moved P4 205.5 mm to (271.0, 28.1), turned to 180 degrees
- moved C21 183.3 mm to (262.2, 52.4), turned to 180 degrees
- moved C19 180.3 mm to (262.2, 54.6), turned to 180 degrees
- moved C20 175.0 mm to (262.2, 44.0), turned to 180 degrees
- moved C22 172.8 mm to (258.4, 48.2), turned to 90 degrees
- moved C18 172.5 mm to (262.2, 60.0), turned to 180 degrees
- moved C23 170.4 mm to (262.2, 46.0)
- moved C8 162.6 mm to (251.8, 52.2), turned to 90 degrees
- moved C4 162.3 mm to (205.8, 29.6), turned to 180 degrees
- moved R7 161.6 mm to (204.6, 27.6), turned to 0 degrees
- moved D3 160.9 mm to (229.2, 16.2)
- moved X2 160.3 mm to (238.6, 55.0)
- moved P1 160.2 mm to (193.0, 17.0), turned to 270 degrees
- moved R22 160.2 mm to (229.2, 20.0)
- moved C15 159.3 mm to (237.6, 55.0)
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Connections:
- C1 pad 1: GND -> Net-(C1-Pad1)
- C1 pad 2: V_SUPPLY -> GND
- C10 pad 2: VCC -> +3V3
- C11 pad 2: VCC -> +3V3
- C12 pad 2: VCC -> +3V3
- C13 pad 2: VCC -> +3V3
- C14 pad 2: VCC -> +3V3
- C18 pad 1: Net-(C18-Pad1) -> /MCU/ADC_TEMP
- C19 pad 1: GND -> /MCU/BR_SO2
- C19 pad 2: Net-(C19-Pad2) -> GND
- C2 pad 1: GND -> +3V3
- C2 pad 2: /MCU/AN_IN -> GND
- C20 pad 1: GND -> /MCU/BR_SO1
- C20 pad 2: Net-(C20-Pad2) -> GND
- C21 pad 1: GND -> /MCU/SENS3
- C21 pad 2: Net-(C21-Pad2) -> GND
- C22 pad 1: Net-(C22-Pad1) -> /MCU/SENS2
- C22 pad 2: Net-(C22-Pad2) -> GND
- C23 pad 1: GND -> /MCU/SENS1
- C23 pad 2: Net-(C23-Pad2) -> GND
- C31 pad 2: VCC -> +3V3
- C35 pad 2: VCC -> +3V3
- C8 pad 2: V_SUPPLY -> /MCU/AN_IN
- C9 pad 2: V_SUPPLY -> +3V3
- P1 pad 1: +5V -> /CAN bus transceiver/CANH
- P1 pad 2: /Filters/TEMP_IN -> /CAN bus transceiver/CANL
- P1 pad 3: /Filters/HALL1_IN -> GND
- P1 pad 4: /Filters/HALL2_IN -> +3V3
- P1 pad 6: GND -> /Filters/HALL2_IN
- P2 pad 1: VCC -> +3V3
- P3 pad 1: +5V -> Net-(C1-Pad1)
- P3 pad 2: VCC -> Net-(P3-Pad2)
- P3 pad 3: GND -> Net-(P3-Pad3)
- P3 pad 4: /MCU/SCK_ADC_EXT -> GND
- P3 pad 5: /MCU/TX_SDA_NSS -> GND
- P3 pad 6: /MCU/RX_SCL_MOSI -> (no net)
- P4 pad 1: V_SUPPLY -> GND
- R103 pad 2: Net-(R103-Pad2) -> Net-(P3-Pad2)
- R104 pad 2: Net-(R104-Pad2) -> Net-(P3-Pad3)
- R11 pad 2: VCC -> +3V3
- R12 pad 2: VCC -> +3V3
- R13 pad 2: VCC -> +3V3
- R22 pad 2: VCC -> +3V3
- R3 pad 1: V_SUPPLY -> /CAN bus transceiver/CANH
- R3 pad 2: /MCU/AN_IN -> /CAN bus transceiver/CANL
- R5 pad 1: /MCU/SERVO -> Net-(P1-Pad16)
- R5 pad 2: Net-(K1-Pad1) -> /MCU/SERVO
- R7 pad 2: VCC -> +3V3
- U1 pad 1: VCC -> +3V3
- U1 pad 13: VCC -> +3V3
- U1 pad 19: VCC -> +3V3
- U1 pad 32: VCC -> +3V3
- U1 pad 48: VCC -> +3V3
- U1 pad 64: VCC -> +3V3
- U2 pad 2: VCC -> +3V3
- U2 pad 3: +5V -> Net-(C1-Pad1)
Routing:
- net GND: track 398.8 -> 0.00 mm, vias 27 -> 0
- net V_SUPPLY: track 290.3 -> 0.00 mm, vias 20 -> 0
- net VCC: track 185.2 -> 0.00 mm, vias 9 -> 0
- net /Mosfet driver/H3_VS: track 166.9 -> 0.00 mm, vias 18 -> 0
- net /Mosfet driver/H1_VS: track 150.6 -> 0.00 mm, vias 17 -> 0
- net /Mosfet driver/H2_VS: track 145.0 -> 0.00 mm, vias 17 -> 0
- net /CAN bus transceiver/CAN_TX: track 3.99 -> 122.9 mm, vias 0 -> 2
- net +5V: track 115.3 -> 0.00 mm, vias 4 -> 0
- net /CAN bus transceiver/CAN_RX: track 12.8 -> 120.4 mm, vias 0 -> 2
- net /MCU/SERVO: track 18.1 -> 111.5 mm, vias 1 -> 2
- net /Filters/TEMP_IN: track 22.4 -> 103.6 mm, vias 0 -> 2
- net /MCU/H1: track 10.1 -> 83.3 mm, vias 2 -> 0
- net /MCU/EN_GATE: track 19.6 -> 92.0 mm
- net /MCU/H2: track 9.02 -> 80.8 mm, vias 0 -> 2
- net /MCU/H3: track 9.22 -> 77.3 mm, vias 0 -> 2
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- removed copper zone on B.Cu, net /Mosfet driver/H1_LOW
- removed copper zone on B.Cu, net /Mosfet driver/H1_VS
- removed copper zone on F.Cu, net /Mosfet driver/H1_VS
- removed copper zone on GND, net /Mosfet driver/H1_VS
- removed copper zone on GND2, net /Mosfet driver/H1_VS
- removed copper zone on B.Cu, net /Mosfet driver/H2_VS
- removed copper zone on F.Cu, net /Mosfet driver/H2_VS
- removed copper zone on GND, net /Mosfet driver/H2_VS
- removed copper zone on GND2, net /Mosfet driver/H2_VS
- removed copper zone on B.Cu, net /Mosfet driver/H3_LOW
- removed copper zone on B.Cu, net /Mosfet driver/H3_VS
- removed copper zone on F.Cu, net /Mosfet driver/H3_VS
- removed copper zone on GND, net /Mosfet driver/H3_VS
- removed copper zone on GND2, net /Mosfet driver/H3_VS
- removed copper zone on B.Cu, net GND
- removed copper zone on F.Cu, net GND
- removed copper zone on GND, net GND
- removed copper zone on GND2, net GND
- removed copper zone on B.Cu, net VCC
- removed copper zone on F.Cu, net V_SUPPLY
Other:
- board size 38.5 x 65 mm -> 100 x 80 mm
- copper layers 4 -> 2
- net class Default: clearance 0.1778 -> 0.2; trace_width 0.2032 -> 0.25; via_dia 0.8 -> 1.8; via_drill 0.5 -> 0.9
- rule trace_clearance: 0.1778 -> 0.2
- rule trace_min: 0.2032 -> 0.2
- rule via_min_drill: 0.5 -> 0.3
- rule via_min_size: 0.8 -> 0.4
- board text removed: "3.3V"
- board text removed: "3.3v"
- board text removed: "5v"
- board text removed: "ADC"
- board text removed: "ADC2"
- board text removed: "Benjamin Vedder"
- board text removed: "CANH"
- board text removed: "CANL"
- board text removed: "CLK"
- board text removed: "DIO"
- board text removed: "GND"
- board text removed: "H1"
- board text removed: "H2"
- board text removed: "H3"
- board text removed: "MISO"
- board text removed: "MOSI"
- board text removed: "NSS"
- board text removed: "RST"
- board text removed: "RX"
- board text removed: "SCK"
- board text removed: "SCL"
- board text removed: "SDA"
- board text removed: "TEMP"
- board text removed: "TX"
- board text removed: "VESC 4.12"
- board text removed: "vedder.se"
