File: board/hall_filters.sch (KiCad schematic (older format))
At the start: 11 parts

Commit message: - changed some more Vcc labels to +3V3 - combined all input connectors into one big connector - changed can transceiver to MAX3051 - removed HV pin from power connector -> divider now on PS board - updated components - startet layout
Parts:
- C4, C5, C6, C7: footprint CRF1:SMD-0603_c -> Capacitors_SMD:C_0805
- R10, R11, R12, R13, R7, R8, R9: footprint CRF1:SMD-0603_r -> Resistors_SMD:R_0805
Connections:
- net labels added: +3V3
- net labels removed: VCC
Changed lines of the file:
@@
 $Descr A4 11693 8268
 encoding utf-8
-Sheet 4 4
+Sheet 3 4
 Title "BLDC Driver 4.11"
 Date "21 aug 2015"
@@
 F 0 "R7" V 4850 3400 50  0000 C CNN
 F 1 "10k" V 4900 3200 50  0000 C CNN
-F 2 "CRF1:SMD-0603_r" H 4900 3200 60  0001 C CNN
+F 2 "Resistors_SMD:R_0805" H 4900 3200 60  0001 C CNN
 F 3 "" H 4900 3200 60  0001 C CNN
 	1    4900 3200
@@
 F 0 "R8" V 5500 3950 50  0000 C CNN
 F 1 "10k" V 5550 3750 50  0000 C CNN
-F 2 "CRF1:SMD-0603_r" H 5550 3750 60  0001 C CNN
+F 2 "Resistors_SMD:R_0805" H 5550 3750 60  0001 C CNN
 F 3 "" H 5550 3750 60  0001 C CNN
 	1    5550 3750
@@
 F 0 "R9" V 5500 3850 50  0000 C CNN
 F 1 "10k" V 5550 3650 50  0000 C CNN
-F 2 "CRF1:SMD-0603_r" H 5550 3650 60  0001 C CNN
+F 2 "Resistors_SMD:R_0805" H 5550 3650 60  0001 C CNN
 F 3 "" H 5550 3650 60  0001 C CNN
 	1    5550 3650
@@
 F 0 "R10" V 5500 3750 50  0000 C CNN
 F 1 "10k" V 5550 3550 50  0000 C CNN
-F 2 "CRF1:SMD-0603_r" H 5550 3550 60  0001 C CNN
+F 2 "Resistors_SMD:R_0805" H 5550 3550 60  0001 C CNN
 F 3 "" H 5550 3550 60  0001 C CNN
 	1    5550 3550
@@
 F 0 "C5" H 6000 4350 50  0000 L CNN
 F 1 "4n7" H 6000 4150 50  0000 L CNN
-F 2 "CRF1:SMD-0603_c" H 5950 4250 60  0001 C CNN
+F 2 "Capacitors_SMD:C_0805" H 5950 4250 60  0001 C CNN
 F 3 "" H 5950 4250 60  0001 C CNN
 	1    5950 4250
@@
 F 0 "C6" H 6250 4350 50  0000 L CNN
 F 1 "4n7" H 6250 4150 50  0000 L CNN
-F 2 "CRF1:SMD-0603_c" H 6200 4250 60  0001 C CNN
+F 2 "Capacitors_SMD:C_0805" H 6200 4250 60  0001 C CNN
 F 3 "" H 6200 4250 60  0001 C CNN
 	1    6200 4250
@@
 F 0 "C7" H 6500 4350 50  0000 L CNN
 F 1 "4n7" H 6500 4150 50  0000 L CNN
-F 2 "CRF1:SMD-0603_c" H 6450 4250 60  0001 C CNN
+F 2 "Capacitors_SMD:C_0805" H 6450 4250 60  0001 C CNN
 F 3 "" H 6450 4250 60  0001 C CNN
 	1    6450 4250
@@
 $EndComp
 $Comp
-L GND-RESCUE-BLDC_4 #PWR030
+L GND-RESCUE-BLDC_4 #PWR046
 U 1 1 53FBB5B2
 P 5950 4450
-F 0 "#PWR030" H 5950 4450 30  0001 C CNN
+F 0 "#PWR046" H 5950 4450 30  0001 C CNN
 F 1 "GND" H 5950 4380 30  0001 C CNN
 F 2 "" H 5950 4450 60  0001 C CNN
@@
 F 0 "R11" V 4950 3400 50  0000 C CNN
 F 1 "2k2" V 5000 3200 50  0000 C CNN
-F 2 "CRF1:SMD-0603_r" H 5000 3200 60  0001 C CNN
+F 2 "Resistors_SMD:R_0805" H 5000 3200 60  0001 C CNN
 F 3 "" H 5000 3200 60  0001 C CNN
 	1    5000 3200
@@
 F 0 "R12" V 5050 3400 50  0000 C CNN
 F 1 "2k2" V 5100 3200 50  0000 C CNN
-F 2 "CRF1:SMD-0603_r" H 5100 3200 60  0001 C CNN
+F 2 "Resistors_SMD:R_0805" H 5100 3200 60  0001 C CNN
 F 3 "" H 5100 3200 60  0001 C CNN
 	1    5100 3200
@@
 F 0 "R13" V 5150 3400 50  0000 C CNN
 F 1 "2k2" V 5200 3200 50  0000 C CNN
-F 2 "CRF1:SMD-0603_r" H 5200 3200 60  0001 C CNN
+F 2 "Resistors_SMD:R_0805" H 5200 3200 60  0001 C CNN
 F 3 "" H 5200 3200 60  0001 C CNN
 	1    5200 3200
@@
 F 0 "C4" H 5150 4350 50  0000 L CNN
 F 1 "4n7" H 5150 4150 50  0000 L CNN
-F 2 "CRF1:SMD-0603_c" H 5100 4250 60  0001 C CNN
+F 2 "Capacitors_SMD:C_0805" H 5100 4250 60  0001 C CNN
 F 3 "" H 5100 4250 60  0001 C CNN
 	1    5100 4250
@@
 $EndComp
 $Comp
-L GND-RESCUE-BLDC_4 #PWR031
+L GND-RESCUE-BLDC_4 #PWR047
 U 1 1 53FBB5D4
 P 5100 4450
-F 0 "#PWR031" H 5100 4450 30  0001 C CNN
+F 0 "#PWR047" H 5100 4450 30  0001 C CNN
 F 1 "GND" H 5100 4380 30  0001 C CNN
 F 2 "" H 5100 4450 60  0001 C CNN
@@
 	1    0    0    -1
 $EndComp
-$Comp
-L VCC #PWR032
-U 1 1 53FBB5DA
-P 4900 2850
-F 0 "#PWR032" H 4900 2950 30  0001 C CNN
-F 1 "VCC" V 4850 2900 30  0000 C CNN
-F 2 "" H 4900 2850 60  0001 C CNN
-F 3 "" H 4900 2850 60  0001 C CNN
-	1    4900 2850
-	1    0    0    -1
-$EndComp
 Connection ~ 5950 3550
 Connection ~ 6200 3650
@@
 	5100 3850 5100 4050
 $Comp
-L GND-RESCUE-BLDC_4 #PWR033
+L GND-RESCUE-BLDC_4 #PWR048
 U 1 1 53FBB5F9
 P 6200 4450
-F 0 "#PWR033" H 6200 4450 30  0001 C CNN
+F 0 "#PWR048" H 6200 4450 30  0001 C CNN
 F 1 "GND" H 6200 4380 30  0001 C CNN
 F 2 "" H 6200 4450 60  0001 C CNN
@@
 $EndComp
 $Comp
-L GND-RESCUE-BLDC_4 #PWR034
+L GND-RESCUE-BLDC_4 #PWR049
 U 1 1 53FBB5FF
 P 6450 4450
-F 0 "#PWR034" H 6450 4450 30  0001 C CNN
+F 0 "#PWR049" H 6450 4450 30  0001 C CNN
 F 1 "GND" H 6450 4380 30  0001 C CNN
 F 2 "" H 6450 4450 60  0001 C CNN
@@
 Connection ~ 4900 3850
 Wire Wire Line
-	4900 2850 4900 2950
+	4900 2750 4900 2950
 Wire Wire Line
 	4900 2850 5200 2850
@@
 Text HLabel 6600 3850 2    60   Output ~ 0
 TEMP_OUT
+$Comp
+L +3V3 #PWR050
+U 1 1 5752258C
+P 4900 2750
+F 0 "#PWR050" H 4900 2600 50  0001 C CNN
+F 1 "+3V3" H 4900 2890 50  0000 C CNN
+F 2 "" H 4900 2750 60  0000 C CNN
+F 3 "" H 4900 2750 60  0000 C CNN
+	1    4900 2750
+	1    0    0    -1
+$EndComp
+Connection ~ 4900 2850
 $EndSCHEMATC
